File: laserDriver.brd (EAGLE design)
At the start: 32.2 x 31.9 mm, 26 parts, among them U1 LED2001, X1 LED_OUT, X2 22-23-2031, X3 FAN_1, X4 FAN_2, X5 FAN_3, X6 FAN_PWM

Commit message: Minor changes.
Routing:
- net N$12: track 26.1 -> 26.7 mm
Changed lines of the file:
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@@
 <?xml version="1.0" encoding="utf-8"?>
 <!DOCTYPE eagle SYSTEM "eagle.dtd">
-<eagle version="7.5.0">
+<eagle version="7.6.0">
 <drawing>
 <settings>
@@
 <layers>
 <layer number="1" name="Top" color="4" fill="1" visible="yes" active="yes"/>
-<layer number="16" name="Bottom" color="1" fill="1" visible="no" active="yes"/>
+<layer number="16" name="Bottom" color="1" fill="1" visible="yes" active="yes"/>
 <layer number="17" name="Pads" color="2" fill="1" visible="yes" active="yes"/>
 <layer number="18" name="Vias" color="2" fill="1" visible="yes" active="yes"/>
@@
 <via x="24.13" y="6.35" extent="1-16" drill="0.35"/>
 <via x="24.13" y="5.08" extent="1-16" drill="0.35"/>
-<via x="24.13" y="16.51" extent="1-16" drill="0.35"/>
-<via x="24.13" y="17.78" extent="1-16" drill="0.35"/>
+<via x="24.892" y="16.256" extent="1-16" drill="0.35"/>
+<via x="24.892" y="17.907" extent="1-16" drill="0.35"/>
 <via x="16.51" y="13.97" extent="1-16" drill="0.35"/>
 <via x="26.67" y="2.54" extent="1-16" drill="0.35"/>
@@
 <via x="7.874" y="20.828" extent="1-16" drill="0.35"/>
 <wire x1="7.874" y1="20.828" x2="16.256" y2="20.828" width="0.3048" layer="16"/>
-<wire x1="16.256" y1="20.828" x2="19.558" y2="17.526" width="0.3048" layer="16"/>
-<via x="19.558" y="17.526" extent="1-16" drill="0.35"/>
-<wire x1="19.558" y1="17.526" x2="19.558" y2="17.592" width="0.3048" layer="1"/>
-<wire x1="19.558" y1="17.592" x2="17.78" y2="19.37" width="0.3048" layer="1"/>
+<wire x1="16.256" y1="20.828" x2="19.431" y2="17.78" width="0.3048" layer="16"/>
+<via x="19.431" y="17.78" extent="1-16" drill="0.35"/>
 <wire x1="7.874" y1="20.828" x2="7.112" y2="20.828" width="0.3048" layer="1"/>
 <wire x1="7.112" y1="20.828" x2="5.842" y2="19.558" width="0.3048" layer="1"/>
 <wire x1="5.842" y1="19.558" x2="3.81" y2="19.558" width="0.3048" layer="1"/>
+<wire x1="19.431" y1="17.78" x2="18.415" y2="17.78" width="0.3" layer="1"/>
+<wire x1="18.415" y1="17.78" x2="17.78" y2="18.415" width="0.3" layer="1"/>
+<wire x1="17.78" y1="18.415" x2="17.78" y2="19.37" width="0.3" layer="1"/>
 </signal>
 <signal name="N$12">
@@
 <wire x1="16.764" y1="23.114" x2="22.098" y2="17.78" width="0.3048" layer="16"/>
 <via x="22.098" y="17.78" extent="1-16" drill="0.35"/>
-<wire x1="22.098" y1="17.78" x2="22.54" y2="17.78" width="0.3048" layer="1"/>
-<wire x1="22.54" y1="17.78" x2="24.13" y2="19.37" width="0.3048" layer="1"/>
 <wire x1="7.874" y1="23.114" x2="6.858" y2="23.114" width="0.3048" layer="1"/>
 <wire x1="6.858" y1="23.114" x2="5.842" y2="22.098" width="0.3048" layer="1"/>
 <wire x1="5.842" y1="22.098" x2="3.81" y2="22.098" width="0.3048" layer="1"/>
+<wire x1="24.13" y1="19.37" x2="24.13" y2="18.288" width="0.3" layer="1"/>
+<wire x1="24.13" y1="18.288" x2="23.622" y2="17.78" width="0.3" layer="1"/>
+<wire x1="23.622" y1="17.78" x2="22.098" y2="17.78" width="0.3" layer="1"/>
 </signal>
 <signal name="N$3">
